Commit message: target fixed

File: dog_gazebo/machine_learning/env/target/target_link.xacro (robot description, xacro)
@@ -1,16 +1,25 @@
 <?xml version="1.0" ?>
-<robot name="tar" xmlns:xacro="http://www.ros.org/wiki/xacro">
-  <link name="base_scan">
+<robot name="target" xmlns:xacro="http://www.ros.org/wiki/xacro">
+  <xacro:include filename="$(find machine_learning)/env/target/target_link.gazebo" />
+  <link name="target_link">
     <collision>
-      <origin xyz="0.005 0.011 0.013" rpy="0 0 0"/> <!--xyz="0.005 0.011 0.013"-->
+      <origin xyz="0 0 0.005" rpy="0 0 0"/> <!--xyz="0.005 0.011 0.013"-->
       <geometry>
-        <box size="0.5 0.5 0.5"/>
+        <box size="0.5 0.5 0.01"/>
       </geometry>
     </collision>
     <visual>
       <geometry>
-        <box size="0.5 0.5 0.5"/>
+        <box size="0.5 0.5 0.01"/>
       </geometry>
     </visual>
+    <inertial>
+      <origin xyz="0 0 0.005" rpy="0 0 0"/>
+      <mass value="0.1"/>
+      <inertia
+          ixx="0.0" ixy="0.0" ixz="0.0"
+          iyy="0.0" iyz="0.0"
+          izz="0.0"/>
+    </inertial>
   </link>
 </robot>

Commit message: fix ubtouchable

File: dog_gazebo/machine_learning/env/target/target_link.xacro (robot description, xacro)
@@ -2,11 +2,6 @@
 <robot name="target" xmlns:xacro="http://www.ros.org/wiki/xacro">
   <xacro:include filename="$(find machine_learning)/env/target/target_link.gazebo" />
+  <static>0</static>
   <link name="target_link">
-    <collision>
-      <origin xyz="0 0 0.005" rpy="0 0 0"/> <!--xyz="0.005 0.011 0.013"-->
-      <geometry>
-        <box size="0.5 0.5 0.01"/>
-      </geometry>
-    </collision>
     <visual>
       <geometry>
