Commit message: depth camara success

File: dog_gazebo/dog2/robots/asus_camera.urdf.xacro (robot description, xacro)
@@ -3,75 +3,4 @@
     <xacro:property name="M_PI" value="3.1415926535897931" />
     <xacro:property name="name" value="Xtion" />
-    <xacro:property name="parent" value="base_scan" />
-    <!--
-     The asus_camera_model macro only adds the model, it does not also add
-     the openni gazebo plugin. See the 'asus_camera' macro below for that
-    -->
-    <xacro:macro name="asus_camera_model" params="name parent *origin">
-      <joint name="${name}_joint" type="fixed">
-        <xacro:insert_block name="origin" />
-        <parent link="${parent}"/>
-        <child link="${name}_link"/>
-      </joint>
-      <link name="${name}_link">
-        <inertial>
-          <mass value="0.200" />
-          <origin xyz="0 0 0" rpy="0 0 0" />
-          <inertia ixx="5.8083e-4" ixy="0" ixz="0" iyy="3.0833e-5" iyz="0" izz="5.9083e-4" />
-        </inertial>
-        <visual>
-          <origin xyz="0 0 0" rpy="0 0 0" />
-          <geometry>
-            <mesh filename="package://dog2/meshes/asus_camera/asus_camera_simple.dae"/>
-          </geometry>
-        </visual>
-       <!--
-       <collision>
-          <origin xyz="0 0 0" rpy="0 0 0" />
-          <geometry>
-            <box size="0.035 0.185 0.025"/>
-          </geometry>
-        </collision>
-        -->
-        <collision>
-          <origin xyz="0 0 0" rpy="0 0 0" />
-          <geometry>
-            <mesh filename="package://dog2/meshes/asus_camera/asus_camera_simple.dae"/>
-          </geometry>
-        </collision>
-      </link>
-      <joint name="${name}_depth_joint" type="fixed">
-        <origin xyz="0.0 0.049 0.0" rpy="0 0 0" />
-        <parent link="${name}_link" />
-        <child link="${name}_depth_frame"/>
-      </joint>
-      <link name="${name}_depth_frame"/>
-      <joint name="${name}_depth_optical_joint" type="fixed">
-        <origin xyz="0 0 0" rpy="${-M_PI/2} 0.0 ${-M_PI/2}" />
-        <parent link="${name}_depth_frame" />
-        <child link="${name}_depth_optical_frame"/>
-      </joint>
-      <link name="${name}_depth_optical_frame"/>
-      <joint name="${name}_rgb_joint" type="fixed">
-        <origin xyz="0.0 0.022 0.0" rpy="0 0 0" />
-        <parent link="${name}_link" />
-        <child link="${name}_rgb_frame"/>
-      </joint>
-      <link name="${name}_rgb_frame"/>
-      <joint name="${name}_rgb_optical_joint" type="fixed">
-        <origin xyz="0 0 0" rpy="${-M_PI/2} 0.0 ${-M_PI/2}" />
-        <parent link="${name}_rgb_frame" />
-        <child link="${name}_rgb_optical_frame"/>
-      </joint>
-      <link name="${name}_rgb_optical_frame"/>
-    </xacro:macro>
-    <!--
-     The asus_camera macro only adds the model, and also adds
-     the openni gazebo plugin.
-    -->
-    <xacro:macro name="asus_camera" params="name parent *origin">
-      <xacro:asus_camera_model name="${name}" parent="${parent}">
-        <xacro:insert_block name="origin" />
-      </xacro:asus_camera_model>
       <!-- ASUS Xtion PRO camera for simulation -->
       <gazebo reference="${name}_depth_frame">
@@ -100,4 +29,3 @@
         </sensor>
       </gazebo>
-    </xacro:macro>
   </robot>

File: dog_gazebo/dog2/robots/dog2.xacro (robot description, xacro)
@@ -3,9 +3,7 @@
   <xacro:property name="cameraSize" value="0.05"/>
   <xacro:property name="cameraMass" value="0.1"/>
-  <xacro:include filename="$(find dog2)/robots/dog1.gazebo" />
+  <xacro:include filename="$(find dog2)/robots/dog2.gazebo" />
   <xacro:include filename="$(find dog2)/robots/materials.xacro" />
-  <xacro:include filename="$(find dog2)/robots/asus_camera.urdf.xacro" />
-  <link
-    name="base_link">
+  <link name="base_link">
     <inertial>
       <origin
@@ -28,5 +26,5 @@
       <geometry>
         <mesh
-          filename="package://dog1/meshes/base_link.STL" />
+          filename="package://dog2/meshes/base_link.STL" />
       </geometry>
       <material
@@ -42,10 +40,9 @@
       <geometry>
         <mesh
-          filename="package://dog1/meshes/base_link.STL" />
-      </geometry>
-    </collision>
-  </link>
-  <link
-    name="L_Link">
+          filename="package://dog2/meshes/base_link.STL" />
+      </geometry>
+    </collision>
+  </link>
+  <link name="L_Link">
     <inertial>
       <origin
@@ -68,5 +65,5 @@
       <geometry>
         <mesh
-          filename="package://dog1/meshes/L_Link.STL" />
+          filename="package://dog2/meshes/L_Link.STL" />
       </geometry>
       <material
@@ -82,5 +79,5 @@
       <geometry>
         <mesh
-          filename="package://dog1/meshes/L_Link.STL" />
+          filename="package://dog2/meshes/L_Link.STL" />
       </geometry>
     </collision>
@@ -102,6 +99,5 @@
   </joint>
   <!--###################################################-->
-  <link
-    name="R_Link">
+  <link name="R_Link">
     <inertial>
       <origin
@@ -124,5 +120,5 @@
       <geometry>
         <mesh
-          filename="package://dog1/meshes/R_Link.STL" />
+          filename="package://dog2/meshes/R_Link.STL" />
       </geometry>
       <material
@@ -138,5 +134,5 @@
       <geometry>
         <mesh
-          filename="package://dog1/meshes/R_Link.STL" />
+          filename="package://dog2/meshes/R_Link.STL" />
       </geometry>
     </collision>
@@ -157,6 +153,5 @@
     <joint_properties damping="0.0" friction="0.0"/>
   </joint>
-  <link
-    name="free_Link">
+  <link name="free_Link">
     <inertial>
       <origin
@@ -179,5 +174,5 @@
       <geometry>
         <mesh
-          filename="package://dog1/meshes/free_Link.STL" />
+          filename="package://dog2/meshes/free_Link.STL" />
       </geometry>
       <material
@@ -193,5 +188,5 @@
       <geometry>
         <mesh
-          filename="package://dog1/meshes/free_Link.STL" />
+          filename="package://dog2/meshes/free_Link.STL" />
       </geometry>
     </collision>
@@ -233,3 +228,22 @@
     <child link="base_scan"/>
   </joint>
+  <link name="asus_link">
+    <visual>
+      <origin xyz="0 0 0" rpy="0 0 0" />
+      <geometry>
+        <mesh filename="package://dog2/meshes/asus_camera/asus_camera_simple.dae"/>
+      </geometry>
+    </visual>
+    <collision>
+      <origin xyz="0 0 0" rpy="0 0 0" />
+      <geometry>
+        <mesh filename="package://dog2/meshes/asus_camera/asus_camera_simple.dae"/>
+      </geometry>
+    </collision>
+  </link>
+  <joint name="asus_depth_joint" type="fixed">
+    <origin xyz="0.2 0 0.05" rpy="0 0 0" />
+    <parent link="base_link" />
+    <child link="asus_link"/>
+  </joint>
 </robot>
